Commit message: incorporated ros2 control urdf into robot description

File: urdf/robot_1.urdf.xacro (robot description, xacro)
@@ -3,4 +3,5 @@
   <!-- Use this if parameters are set from the launch file, otherwise delete -->
   <xacro:arg name="prefix" default="" />
+  <xacro:include filename="$(find tutorial_robot_1)/urdf/robot_1/robot_1_macro.ros2_control.xacro"/>
   <xacro:include filename="$(find tutorial_robot_1)/urdf/robot_1/robot_1_macro.xacro"/>
   <!-- create link fixed to the "world" -->
@@ -9,5 +10,5 @@
   <!-- set prefix if multiple robots are used -->
   <xacro:robot_1 prefix="$(arg prefix)" parent="world" >
-    <origin xyz="0 0 0" rpy="0 0 0" />          <!-- position robot in the world -->
+    <origin xyz="0 0 0.05" rpy="0 0 0" />          <!-- position robot in the world -->
   </xacro:robot_1>
 </robot>

File: urdf/robot_1/robot_1_macro.ros2_control.xacro (robot description, xacro)
@@ -1,138 +1,29 @@
 <?xml version="1.0" encoding="UTF-8"?>
 <robot xmlns:xacro="http://wiki.ros.org/xacro">
-  <xacro:macro name="robot_1_ros2_control" params="
-               name
-               prefix
-               use_mock_hardware:=^|false
-               mock_sensor_commands:=^|false
-               sim_gazebo_classic:=^|false
-               sim_gazebo:=^|false
-               simulation_controllers"
-               >
-    <ros2_control name="${name}" type="system">
-      <hardware>
-        <xacro:if value="${use_mock_hardware}">
-          <plugin>mock_components/GenericSystem</plugin>
-          <param name="mock_sensor_commands">${mock_sensor_commands}</param>
-        </xacro:if>
-        <xacro:if value="${sim_gazebo_classic}">
-          <plugin>gazebo_ros2_control/GazeboSystem</plugin>
-        </xacro:if>
-        <xacro:if value="${sim_gazebo}">
-          <plugin>ign_ros2_control/IgnitionSystem</plugin>
-        </xacro:if>
-        <xacro:unless value="${use_mock_hardware or sim_gazebo_classic or sim_gazebo}">
-          <plugin>robot_hardware_inteface/RobotHardwareInteface</plugin>
-        </xacro:unless>
-      </hardware>
-      <joint name="${prefix}joint1">
-        <command_interface name="position">     <!-- Add/Remove interfaces as needed -->
-          <param name="min">-1</param>
-          <param name="max">1</param>
-        </command_interface>
-        <state_interface name="position">
-          <param name="initial_value">0.0</param>
-        </state_interface>
-        <state_interface name="velocity"/>
-        <state_interface name="acceleration"/>
-      </joint>
-      <joint name="${prefix}joint2">
-        <command_interface name="position">     <!-- Add/Remove interfaces as needed -->
-          <param name="min">-1</param>
-          <param name="max">1</param>
-        </command_interface>
-        <state_interface name="position">
-          <param name="initial_value">0.0</param>
-        </state_interface>
-        <state_interface name="velocity"/>
-        <state_interface name="acceleration"/>
-      </joint>
-      <joint name="${prefix}joint3">
-        <command_interface name="position">     <!-- Add/Remove interfaces as needed -->
-          <param name="min">-1</param>
-          <param name="max">1</param>
-        </command_interface>
-        <state_interface name="position">
-          <param name="initial_value">0.0</param>
-        </state_interface>
-        <state_interface name="velocity"/>
-        <state_interface name="acceleration"/>
-      </joint>
-      <joint name="${prefix}joint4">
-        <command_interface name="position">     <!-- Add/Remove interfaces as needed -->
-          <param name="min">-1</param>
-          <param name="max">1</param>
-        </command_interface>
-        <state_interface name="position">
-          <param name="initial_value">0.0</param>
-        </state_interface>
-        <state_interface name="velocity"/>
-        <state_interface name="acceleration"/>
-      </joint>
-      <joint name="${prefix}joint5">
-        <command_interface name="position">     <!-- Add/Remove interfaces as needed -->
-          <param name="min">-1</param>
-          <param name="max">1</param>
-        </command_interface>
-        <state_interface name="position">
-          <param name="initial_value">0.0</param>
-        </state_interface>
-        <state_interface name="velocity"/>
-        <state_interface name="acceleration"/>
-      </joint>
-      <joint name="${prefix}joint6">
-        <command_interface name="position">     <!-- Add/Remove interfaces as needed -->
-          <param name="min">-1</param>
-          <param name="max">1</param>
-        </command_interface>
-        <state_interface name="position">
-          <param name="initial_value">0.0</param>
-        </state_interface>
-        <state_interface name="velocity"/>
-        <state_interface name="acceleration"/>
-      </joint>
-      <sensor name="tcp_fts_sensor">            <!-- Remove/change sensors as needed -->
-        <state_interface name="fx"/>
-        <state_interface name="fy"/>
-        <state_interface name="fz"/>
-        <state_interface name="tx"/>
-        <state_interface name="ty"/>
-        <state_interface name="tz"/>
-        <param name="frame_id">tool0</param>    <!-- Change sensors as needed -->
-        <param name="min_fx">-100</param>
-        <param name="max_fx">100</param>
-        <param name="min_fy">-100</param>
-        <param name="max_fy">100</param>
-        <param name="min_fz">-200</param>
-        <param name="max_fz">200</param>
-        <param name="min_tx">-10</param>
-        <param name="max_tx">10</param>
-        <param name="min_ty">-10</param>
-        <param name="max_ty">10</param>
-        <param name="min_tz">-15</param>
-        <param name="max_tz">15</param>
-      </sensor>
-    </ros2_control>
-    <xacro:if value="$(arg sim_gazebo_classic)">
-      <!-- Gazebo plugins -->
-      <gazebo reference="world">
-      </gazebo>
-      <gazebo>
-        <plugin filename="libgazebo_ros2_control.so" name="gazebo_ros2_control">
-          <parameters>${simulation_controllers}</parameters>
-        </plugin>
-      </gazebo>
-    </xacro:if>
-    <xacro:if value="$(arg sim_gazebo)">
-      <!-- Gazebo plugins -->
-      <gazebo reference="world">
-      </gazebo>
-      <gazebo>
-        <plugin filename="libign_ros2_control-system.so" name="ign_ros2_control::IgnitionROS2ControlPlugin">
-          <parameters>${simulation_controllers}</parameters>
-          <controller_manager_node_name>${prefix}controller_manager</controller_manager_node_name>
-        </plugin>
-      </gazebo>
-    </xacro:if>
-  </xacro:macro>
+  <ros2_control name="robot_1" type="system">
+    <hardware>
+      <plugin>gazebo_ros2_control/GazeboSystem</plugin>
+    </hardware>
+    <joint name="left_wheel_joint">
+      <command_interface name="velocity">
+        <param name="min">-10</param>
+        <param name="max">10</param>
+      </command_interface>
+      <state_interface name="velocity"/>
+      <state_interface name="position"/>
+    </joint>
+    <joint name="right_wheel_joint">
+      <command_interface name="velocity">
+        <param name="min">-10</param>
+        <param name="max">10</param>
+      </command_interface>
+      <state_interface name="velocity"/>
+      <state_interface name="position"/>
+    </joint>
+  </ros2_control>
+  <gazebo>
+    <plugin name="gazebo_ros2_control" filename="libgazebo_ros2_control.so">
+      <parameters>$(find tutorial_robot_1)/config/robot_1_controllers.yaml</parameters>
+    </plugin>
+  </gazebo>
 </robot>

File: urdf/robot_1/robot_1_macro.xacro (robot description, xacro)
@@ -15,9 +15,4 @@
     </joint>
     <!-- CHASSIS LINK -->
-    <joint name="${prefix}chassis_joint" type="fixed">
-      <parent link="${prefix}base_link"/>
-      <child link="${prefix}chassis_link"/>
-      <origin xyz="-0.1 0 0"/>
-    </joint>
     <link name="${prefix}chassis_link">
       <visual>
@@ -38,11 +33,13 @@
       </xacro:box_inertial>
     </link>
+    <joint name="${prefix}chassis_joint" type="fixed">
+      <parent link="${prefix}base_link"/>
+      <child link="${prefix}chassis_link"/>
+      <origin xyz="-0.1 0 0"/>
+    </joint>
+    <gazebo reference="chassis_link">
+      <material>Gazebo/Turquoise</material>
+    </gazebo>
     <!-- LEFT WHEEL LINK-->
-    <joint name="${prefix}left_wheel_joint" type="continuous">
-      <parent link="${prefix}base_link"/>
-      <child link="${prefix}left_wheel_link"/>
-      <origin xyz="0 0.15 0" rpy="${-pi/2} 0 0"/>
-      <axis xyz="0 0 1"/>
-    </joint>
     <link name="${prefix}left_wheel_link">
       <visual>
@@ -61,11 +58,14 @@
       </collision>
     </link>
+    <joint name="${prefix}left_wheel_joint" type="continuous">
+      <parent link="${prefix}base_link"/>
+      <child link="${prefix}left_wheel_link"/>
+      <origin xyz="0 0.15 0" rpy="${-pi/2} 0 0"/>
+      <axis xyz="0 0 1"/>
+    </joint>
+    <gazebo reference="left_wheel_link">
+      <material>Gazebo/White</material>
+    </gazebo>
     <!-- RIGHT WHEEL LINK-->
-    <joint name="${prefix}right_wheel_joint" type="continuous">
-      <parent link="${prefix}base_link"/>
-      <child link="${prefix}right_wheel_link"/>
-      <origin xyz="0 -0.15 0" rpy="${pi/2} 0 0"/>
-      <axis xyz="0 0 -1"/>
-    </joint>
     <link name="${prefix}right_wheel_link">
       <visual>
@@ -84,10 +84,14 @@
       </collision>
     </link>
+    <joint name="${prefix}right_wheel_joint" type="continuous">
+      <parent link="${prefix}base_link"/>
+      <child link="${prefix}right_wheel_link"/>
+      <origin xyz="0 -0.15 0" rpy="${pi/2} 0 0"/>
+      <axis xyz="0 0 -1"/>
+    </joint>
+    <gazebo reference="right_wheel_link">
+      <material>Gazebo/White</material>
+    </gazebo>
     <!-- CASTER WHEEL LINK -->
-    <joint name="${prefix}caster_wheel_joint" type="fixed">
-      <parent link="${prefix}chassis_link"/>
-      <child link="${prefix}caster_wheel_link"/>
-      <origin xyz="0.24 0 0"/>
-    </joint>
     <link name="${prefix}caster_wheel_link">
       <visual>
@@ -105,4 +109,12 @@
       </collision>
     </link>
+    <joint name="${prefix}caster_wheel_joint" type="fixed">
+      <parent link="${prefix}chassis_link"/>
+      <child link="${prefix}caster_wheel_link"/>
+      <origin xyz="0.24 0 0"/>
+    </joint>
+    <gazebo reference="caster_wheel_link">
+      <material>Gazebo/Red</material>
+    </gazebo>
   </xacro:macro>
 </robot>

Commit message: fixed tf2 frame hierarchy

File: urdf/robot_1.urdf.xacro (robot description, xacro)
@@ -5,10 +5,8 @@
   <xacro:include filename="$(find tutorial_robot_1)/urdf/robot_1/robot_1_macro.ros2_control.xacro"/>
   <xacro:include filename="$(find tutorial_robot_1)/urdf/robot_1/robot_1_macro.xacro"/>
-  <!-- create link fixed to the "world" -->
-  <link name="world" />
   <!-- Load robot's macro with parameters -->
   <!-- set prefix if multiple robots are used -->
-  <xacro:robot_1 prefix="$(arg prefix)" parent="world" >
-    <origin xyz="0 0 0.05" rpy="0 0 0" />          <!-- position robot in the world -->
+  <xacro:robot_1 prefix="$(arg prefix)">
+    <origin xyz="0 0 0" rpy="0 0 0" />          <!-- position robot in the world -->
   </xacro:robot_1>
 </robot>

File: urdf/robot_1/robot_1_macro.xacro (robot description, xacro)
@@ -2,16 +2,8 @@
 <robot xmlns:xacro="http://wiki.ros.org/xacro">
   <xacro:include filename="$(find tutorial_robot_1)/urdf/common.xacro" />
-  <xacro:macro name="robot_1" params="prefix parent *origin">
+  <xacro:macro name="robot_1" params="prefix *origin">
     <!-- BASE LINK -->
     <link name="${prefix}base_link">
-      <!-- Default inertial for Gazebo/Ingnition - copy and edit block from 'common.xacro'
-           to get more realistic behaviour-->
-      <xacro:default_inertial/>
     </link>
-    <joint name="${prefix}base_joint" type="fixed">
-      <xacro:insert_block name="origin" />
-      <parent link="${parent}" />
-      <child link="${prefix}base_link" />
-    </joint>
     <!-- CHASSIS LINK -->
     <link name="${prefix}chassis_link">
@@ -116,4 +108,6 @@
     <gazebo reference="caster_wheel_link">
       <material>Gazebo/Red</material>
+        <mu1 value="0.001"/>
+        <mu2 value="0.001"/>
     </gazebo>
   </xacro:macro>
